File: PCB/voxid.kicad_sch (KiCad schematic)
At the start: 50 parts, among them J1 Conn_01x02_Pin, J2 Conn_01x02_Pin, J3 Conn_01x02_Pin, J4 v3.3, J5 v3.3, J6 AudioOut, J7 Conn_01x02_Pin, U1 TL072, U2 TL072, U3 TL072, U4 LM1117T-3.3

Commit message: wip: Actualizacion de PCB y simulaciones
Connections:
- net LPF: now reaches J1.1 (Pin_1), R9.2
- net Sound: now reaches C6.1, J7.1 (Pin_1)
- net HPF: now reaches J3.1 (Pin_1), RV5.1, RV5.2
Other:
- moved on the sheet: C1, C10, C17, C2, C3, C4, C5, C6, C7, C8, C9, Cin1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

Commit message: feat: Actualizar diseño PCB y agregar diagrama del sistema
Parts:
- removed C17: 100nF, Capacitor_THT:CP_Radial_Tantal_D5.0mm_P5.00mm, symbol Device:C
- removed C5: 10nF, Capacitor_THT:CP_Radial_Tantal_D5.0mm_P5.00mm, symbol Device:C
- removed Cin1: 1uF, Capacitor_THT:CP_Radial_Tantal_D5.0mm_P5.00mm, symbol Device:C
- removed J5: v3.3, Connector_PinHeader_2.54mm:PinHeader_1x02_P2.54mm_Vertical, symbol Connector:Conn_01x02_Pin
- removed R11: 1k, Resistor_THT:R_Axial_DIN0309_L9.0mm_D3.2mm_P12.70mm_Horizontal, symbol Device:R
- removed R12: 2.2k, Resistor_THT:R_Axial_DIN0309_L9.0mm_D3.2mm_P12.70mm_Horizontal, symbol Device:R
- removed R13, R7, R8, R9: 10k, Resistor_THT:R_Axial_DIN0309_L9.0mm_D3.2mm_P12.70mm_Horizontal, symbol Device:R
- removed RV1: 17.2k, Potentiometer_THT:Potentiometer_Bourns_3296W_Vertical, symbol Device:R_Potentiometer
- removed RV2: 41.2k, Potentiometer_THT:Potentiometer_Bourns_3296W_Vertical, symbol Device:R_Potentiometer
- removed RV3: 6.04k, Potentiometer_THT:Potentiometer_Bourns_3296W_Vertical, symbol Device:R_Potentiometer
- removed RV4: 14.7k, Potentiometer_THT:Potentiometer_Bourns_3296W_Vertical, symbol Device:R_Potentiometer
- removed RV5, RV6: 2.43k, Potentiometer_THT:Potentiometer_Bourns_3296W_Vertical, symbol Device:R_Potentiometer
- removed RV7, RV8: 1.02k, Potentiometer_THT:Potentiometer_Bourns_3296W_Vertical, symbol Device:R_Potentiometer
- removed RV9: 100, Potentiometer_THT:Potentiometer_Bourns_3296W_Vertical, symbol Device:R_Potentiometer
- added C6: 27nF, Capacitor_THT:CP_Radial_Tantal_D5.0mm_P5.00mm, symbol Device:C
- added Caudio1: 1uF, Capacitor_THT:CP_Radial_Tantal_D5.0mm_P5.00mm, symbol Device:C
- added Cref1: 22uF, Capacitor_THT:CP_Radial_Tantal_D5.0mm_P5.00mm, symbol Device:C
- added R1: 1.3k, Resistor_THT:R_Axial_DIN0411_L9.9mm_D3.6mm_P12.70mm_Horizontal, symbol Device:R
- added R10: 779, Resistor_THT:R_Axial_DIN0411_L9.9mm_D3.6mm_P12.70mm_Horizontal, symbol Device:R
- added R14: 1.67.k, Resistor_THT:R_Axial_DIN0411_L9.9mm_D3.6mm_P12.70mm_Horizontal, symbol Device:R
- added R15: 2.2k, Resistor_THT:R_Axial_DIN0411_L9.9mm_D3.6mm_P12.70mm_Horizontal, symbol Device:R
- added R16: 1k, Resistor_THT:R_Axial_DIN0411_L9.9mm_D3.6mm_P12.70mm_Horizontal, symbol Device:R
- added R17, R18, R19, R20, R21: 10k, Resistor_THT:R_Axial_DIN0411_L9.9mm_D3.6mm_P12.70mm_Horizontal, symbol Device:R
- added R2: 8.87k, Resistor_THT:R_Axial_DIN0411_L9.9mm_D3.6mm_P12.70mm_Horizontal, symbol Device:R
- added R3: 3.09k, Resistor_THT:R_Axial_DIN0411_L9.9mm_D3.6mm_P12.70mm_Horizontal, symbol Device:R
- added R4: 3.65k, Resistor_THT:R_Axial_DIN0411_L9.9mm_D3.6mm_P12.70mm_Horizontal, symbol Device:R
- added R5: 1.64k, Resistor_THT:R_Axial_DIN0411_L9.9mm_D3.6mm_P12.70mm_Horizontal, symbol Device:R
- C1: renamed from C6; value 100nF -> 470nF
- C2: value 12nF -> 470nF
- C3: value 10nF -> 470nF
- C4: value 68nF -> 470nF
- C7: value 100nF -> 2.7nF
- C8: value 100nF -> 27nF
- C9: value 100nF -> 20nF
- Cout1: renamed from C10; value 100nF -> 10uF
- J1: renamed from J7; value Conn_01x02_Pin -> Audio
- J2: renamed from J3; value Conn_01x02_Pin -> HPF_O
- J3: renamed from J1; value Conn_01x02_Pin -> LPFO
- J4: renamed from J2; value Conn_01x02_Pin -> Offset
- R22: renamed from R5; value 10k -> 1.05K; footprint Resistor_THT:R_Axial_DIN0309_L9.0mm_D3.2mm_P12.70mm_Horizontal -> Resistor_THT:R_Axial_DIN0411_L9.9mm_D3.6mm_P12.70mm_Horizontal
- R23: renamed from R4; value 10k -> 1k; footprint Resistor_THT:R_Axial_DIN0309_L9.0mm_D3.2mm_P12.70mm_Horizontal -> Resistor_THT:R_Axial_DIN0411_L9.9mm_D3.6mm_P12.70mm_Horizontal
- R6: value 10k -> 5.87k; footprint Resistor_THT:R_Axial_DIN0309_L9.0mm_D3.2mm_P12.70mm_Horizontal -> Resistor_THT:R_Axial_DIN0411_L9.9mm_D3.6mm_P12.70mm_Horizontal
- renumbered C1 to Cin1, J4 to J5, RV10 to RV1, TP01 to TP1
Connections:
- net +3.3V: now also R15.1
- net GND: now also C7.1, C9.1, Cref1.1, R2.2, R21.2, R4.2; no longer C3.2
- net HPF: now also R5.1
- net LPF: now also R18.1
- net Vref: now also R22.2, R23.1, Cref1.2
- net at C1.2: now also C2.1, R1.1; no longer C7.1
- net at C7.2: now also R6.2, U2.3 (+); no longer U1.5 (+)
- net at MK1.2 (+): now also Caudio1.1, R15.2
- net at J3.2 (Pin_2), U3.1, U3.2 (-): now also C8.2; no longer C4.2
- net at C4.1: now also C3.2, R3.1
- net at RV1.1, RV1.2: now also R17.2
- net at U1.2 (-): now also R16.2, R17.1
- net at U1.6 (-), U1.7: now also C3.1, R1.2; no longer C8.1
- net at U2.1, U2.2 (-): now also C6.2, R10.1; no longer C2.2
- net at J4.2 (Pin_2): now also R20.1
- net at J6.1 (Pin_1), U3.7: now also R19.2; no longer R6.1
- net at U3.6 (-): now also R18.2, R19.1; no longer R6.2
- net at U3.3 (+): now also C9.2, R14.2
- net at U3.5 (+): now also R20.2, R21.1
- net at U2.5 (+): now also C4.2, R4.1; no longer C9.2
- net at J2.2 (Pin_2), U2.6 (-), U2.7: now also R3.2
- new net: Caudio1.2, R16.1
- new net: C8.1, R10.2, R14.1
- new net: C2.2, R2.1, U1.5 (+)
- new net: C6.1, R5.2, R6.1
Other:
- moved on the sheet: J3, J5, TP1, TP2, TP3, U2A, U3A

Commit message: pcb: Incluir proteccion del ADC
Parts:
- added D1, D2: 1N5819, Diode_THT:D_DO-41_SOD81_P10.16mm_Horizontal, symbol Diode:1N5819
- added Rlim1: 4.7k, Resistor_THT:R_Axial_DIN0411_L9.9mm_D3.6mm_P12.70mm_Horizontal, symbol Device:R
- C6, C8: value 27nF -> 22nF
- C7: value 2.7nF -> 2.2nF
- C9: value 20nF -> 10nF
- R1: value 1.3k -> 1.2k
- R10: value 779 -> 820
- R14: value 1.67.k -> 3.9k
- R2: value 8.87k -> 8.2k
- R3: value 3.09k -> 3.3k
- R4: value 3.65k -> 3.9k
- R5: value 1.64k -> 2.2k
- R6: value 5.87k -> 6.8k
Connections:
- net +3.3V: now also D1.1 (K)
- net GND: now also D2.2 (A)
- net S: now reaches R19.2, U3.7
- net S: now also Rlim1.1; no longer J6.1 (Pin_1)
- new net: D1.2 (A), D2.1 (K), J6.1 (Pin_1), Rlim1.2
Other:
- moved on the sheet: Cref1

Commit message: pcb: Creacion de geber para cnc
Parts:
- added Cref2, Cref3, Cref4, Cref5, Cref6, Cref7: 100nF, Capacitor_THT:CP_Radial_Tantal_D5.0mm_P5.00mm, symbol Device:C
- added J7: v3.3, Connector_PinHeader_2.54mm:PinHeader_1x02_P2.54mm_Vertical, symbol Connector:Conn_01x02_Pin
Connections:
- net +12V: now also Cref4.1, Cref5.2, Cref6.1
- net -12V: now also Cref2.1, Cref3.2, Cref7.1
- net GND: now also Cref2.2, Cref3.1, Cref4.2, Cref5.1, Cref6.2, Cref7.2, J7.2 (Pin_2)
- net at D1.2 (A), D2.1 (K), J6.1 (Pin_1)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: now also J7.1 (Pin_1)
Other:
- moved on the sheet: D1, D2

Commit message: pcb: Pcb lista :)
Parts:
- added J8: Offset, Connector_PinHeader_2.54mm:PinHeader_1x02_P2.54mm_Vertical, symbol Connector:Conn_01x02_Pin
- R1, R10, R14, R15, R16, R17, R18, R19, R2, R20, R21, R22, R23, R3, R4, R5, R6, Rlim1: footprint Resistor_THT:R_Axial_DIN0411_L9.9mm_D3.6mm_P12.70mm_Horizontal -> Resistor_THT:R_Axial_DIN0207_L6.3mm_D2.5mm_P7.62mm_Horizontal
Connections:
- net +3.3V: now also J8.2 (Pin_2); no longer D1.1 (K)
- new net: D1.1 (K), J8.1 (Pin_1)
Other:
- moved on the sheet: D1, D2, J6, J7, Rlim1

Commit message: pcb: ahora si, pcb lista e imagen de la pcb agregada a DOC
Parts:
- removed R22: 1.05K, Resistor_THT:R_Axial_DIN0207_L6.3mm_D2.5mm_P7.62mm_Horizontal, symbol Device:R
- added J9: v3.3, Connector_PinHeader_2.54mm:PinHeader_1x02_P2.54mm_Vertical, symbol Connector:Conn_01x02_Pin
- added RV2: 1.05k, Potentiometer_THT:Potentiometer_Bourns_3296W_Vertical, symbol Device:R_Potentiometer
Connections:
- net GND: now also J9.1 (Pin_1), J9.2 (Pin_2), RV2.1, RV2.2
- net Vref: now also RV2.3
